File: splinktegrated.kicad_pcb (KiCad board)
At the start: 2 copper layers, 41.8 x 68.6 mm, 64 parts, among them J1 USB_C_Receptacle_USB2.0, J10 Ribbon, J11 Serial, J12 Conn_01x04_Female, J13 Conn_01x02_Female, J2 Conn_01x04_Female, J3 Conn_01x04_Female, J4 Conn_01x04_Female, J5 Conn_01x02, J6 Serial, J7 trackball, J8 Ribbon, J9 RGB, SW1 SW_SPST, SW2 SW_SPST, U1 RP2040, U2 USBLC6-2P6, U3 XC6210B332MR-G, U4 USBLC6-2P6, U5 W25Q128JVS, Y1 Crystal_GND24

Commit message: minor changes
Parts:
- removed JP1, JP2: Jumper_2_Open, local-libraries:SolderJumper-2_P1.3mm_Open_RoundedPad1.0x1.5mm
- added J14: USB_C_Receptacle_USB2.0, Connector_USB:USB_C_Receptacle_HRO_TYPE-C-31-M-12, B.Cu at (151.4, 137.7)
- J1: footprint drawings:GT-USB-7014C -> Connector_USB:USB_C_Receptacle_HRO_TYPE-C-31-M-12
- J11: value Serial -> RJ9; footprint drawings:Jack_3.5mm_PJ320E_Horizontal_custom -> JohnDeereLibrary:AMPHENOL_73306-111LF; moved to B.Cu
- J6: value Serial -> RJ9; footprint drawings:Jack_3.5mm_PJ320E_Horizontal_custom -> JohnDeereLibrary:AMPHENOL_73306-111LF; moved to F.Cu
- moved J6 16.5 mm to (122.7, 81.7), turned to 90 degrees
- moved J11 12.2 mm to (122.6, 81.7), turned to 90 degrees
- moved J1 3.22 mm to (151.4, 137.7)
Connections:
- U1 pad 3: serial_l -> unconnected-(U1-GPIO1-Pad3)
- U1 pad 4: unconnected-(U1-GPIO2-Pad4) -> I2C1 SDA
- U1 pad 5: unconnected-(U1-GPIO3-Pad5) -> I2C1 SCL
- U2 pad 1: serial_l -> I2C1 SCL Raw
- U2 pad 3: unconnected-(U2-I/O2-Pad3) -> I2C1 SDA Raw
- U2 pad 4: unconnected-(U2-I/O2-Pad4) -> I2C1 SDA
- U2 pad 6: serial_l -> I2C1 SCL
Routing:
- net serial_l: track 40.1 -> 0.00 mm, vias 2 -> 0
- net +3V3: track 106.8 -> 92.3 mm, vias 3 -> 2
- net unconnected-(U1-GPIO1-Pad3): track 0.00 -> 7.28 mm, vias 0 -> 1
- net Net-(JP1-A): track 5.68 -> 0.00 mm
- net GND: track 42.4 -> 37.8 mm
- net Net-(J1-SHIELD): track 4.25 -> 8.32 mm
- net Net-(JP2-A): track 3.68 -> 0.00 mm
Other:
- outline, holes or cut-outs redrawn

Commit message: major work done. outline finished
Parts:
- removed J14: USB_C_Receptacle_USB2.0, Connector_USB:USB_C_Receptacle_HRO_TYPE-C-31-M-12
- moved kibuzzard-61F01C84 19.2 mm to (115.6, 93.9)
- moved J11 13.3 mm to (135.9, 80.3)
- moved J6 13.3 mm to (135.9, 80.3)
- moved R11 12.5 mm to (154.3, 79.5), turned to 0 degrees
- moved U2 11.9 mm to (135.9, 93.8)
- moved R10 11.6 mm to (156.5, 79.5), turned to 0 degrees
- moved C1 10.8 mm to (148.3, 82.0), turned to -90 degrees
- moved U3 6.56 mm to (151.3, 82.1), turned to -90 degrees
- moved SW2 6.11 mm to (134.6, 101.6)
- moved SW1 6.07 mm to (134.6, 101.6)
- moved C2 5.12 mm to (150.9, 85.1), turned to 180 degrees
- moved D2 4.17 mm to (154.4, 82.1), turned to -90 degrees
- moved F1 4.14 mm to (156.6, 82.1), turned to -90 degrees
- moved C7 3.20 mm to (148.9, 90.9), turned to 180 degrees
- moved C10 2.75 mm to (140.5, 92.2), turned to -90 degrees
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Routing:
- net GND: track 37.8 -> 18.4 mm, vias 24 -> 23
- net /VBUS_DET: track 13.7 -> 32.0 mm
- net +3V3: track 92.3 -> 108.0 mm, vias 2 -> 5
- net I2C1 SDA: track 0.00 -> 15.5 mm, vias 0 -> 2
- net I2C1 SCL: track 0.00 -> 13.9 mm, vias 0 -> 2
- net Net-(J1-SHIELD): track 8.32 -> 21.1 mm
- net VBUS: track 31.8 -> 20.9 mm, vias 3 -> 0
- net unconnected-(U1-GPIO1-Pad3): track 7.28 -> 0.00 mm, vias 1 -> 0
- net col6_l: track 39.2 -> 33.3 mm
- net row5_l: track 41.3 -> 35.4 mm
- net col5_l: track 36.8 -> 31.1 mm
- net col4_l: track 34.4 -> 28.9 mm
- net miso_l: track 51.6 -> 46.5 mm
- net row3_l: track 31.6 -> 26.8 mm
- net I2C1 SCL Raw: track 0.00 -> 4.74 mm
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Other:
- outline, holes or cut-outs redrawn

Commit message: USB daugherboard
Parts:
- removed D2: B5817, Diode_SMD:D_SOD-323
- removed F1: Polyfuse, Fuse:Fuse_0603_1608Metric
- removed J12, J4: Conn_01x04_Female, drawings:PinHeader_1x04_P2.54mm_Vertical
- added H1: MountingHole, MountingHole:MountingHole_2.2mm_M2, F.Cu at (199.5, 80.5)
- added H2: MountingHole, MountingHole:MountingHole_2.2mm_M2, F.Cu at (199.5, 92.8)
- added H3: MountingHole, MountingHole:MountingHole_2.2mm_M2, F.Cu at (213.4, 92.8)
- added H4: MountingHole_Pad, MountingHole:MountingHole_2.2mm_M2_Pad, F.Cu at (213.4, 80.5)
Connections:
- R10 pad 2: VBUS -> +5V
Routing:
- net VBUS: track 20.9 -> 0.00 mm
- net (no net): track 0.00 -> 17.6 mm
- net Net-(D2-A): track 2.32 -> 0.00 mm
