File: splinktegrated.kicad_sch (KiCad schematic)
At the start: 52 parts, among them J1 USB_C_Receptacle_USB2.0, J10 Ribbon, J11 Serial, J12 Conn_01x04_Female, J13 Conn_01x02_Female, J2 Conn_01x04_Female, J3 Conn_01x04_Female, J4 Conn_01x04_Female, J5 Conn_01x02, J6 Serial, J7 trackball, J8 Ribbon, J9 RGB, SW1 SW_SPST, SW2 SW_SPST, U1 RP2040, U2 USBLC6-2P6, U3 XC6210B332MR-G, U4 USBLC6-2P6, U5 W25Q128JVS, Y1 Crystal_GND24

Commit message: start to replace audio jacks with rj9s
Parts:
- removed J11, J6: Serial, drawings:Jack_3.5mm_PJ320E_Horizontal_custom, symbol Connector:AudioJack4
- removed JP1, JP2: Jumper_2_Open, local-libraries:SolderJumper-2_P1.3mm_Open_RoundedPad1.0x1.5mm, symbol Jumper:Jumper_2_Open
- added J11, J6: RJ9, JohnDeereLibrary:AMPHENOL_73306-111LF, symbol Connector:RJ9
- added J14: USB_C_Receptacle_USB2.0, Connector_USB:USB_C_Receptacle_HRO_TYPE-C-31-M-12, symbol Connector:USB_C_Receptacle_USB2.0
- J1: footprint drawings:GT-USB-7014C -> Connector_USB:USB_C_Receptacle_HRO_TYPE-C-31-M-12
Connections:
- net D+_daughter: now also J14.A6 (D+), J14.B6 (D+)
- net D-_daughter: now also J14.A7 (D-), J14.B7 (D-)
- net Gnd_daughter: now also J14.A1 (GND), J14.A12 (GND), J14.B1 (GND), J14.B12 (GND)
- net Vbus_daughter: now also J14.A4 (VBUS), J14.A9 (VBUS), J14.B4 (VBUS), J14.B9 (VBUS)
- net serial_l: no longer U1.3 (GPIO1), U2.1 (I/O1), U2.6 (I/O1)
- net I2C1 SDA: now reaches U1.4 (GPIO2)
- net I2C1 SCL: now reaches U1.5 (GPIO3)
- net at J1.A5 (CC1), R4.1: now also J14.A5 (CC1)
- net at J1.B5 (CC2), R5.1: now also J14.B5 (CC2)
- net at FB1.2, J1.S1 (SHIELD): now also J14.S1 (SHIELD)
- new net: U2.1 (I/O1), U2.6 (I/O1)
- no-connect marks 18 -> 14

Commit message: minor changes
Connections:
- net +3V3: now also J11.1, J6.1
- net GND: now also J11.4, J6.4
- net I2C1 SCL: now also U2.6 (I/O1)
- net I2C1 SDA: now also U2.4 (I/O2)
- net I2C1 SCL Raw: now reaches J11.2
- net I2C1 SCL Raw: now also J6.2, U2.1 (I/O1)
- net I2C1 SDA Raw: now reaches J11.3
- net I2C1 SDA Raw: now also J6.3, U2.3 (I/O2)
- no-connect marks 14 -> 12
Other:
- moved on the sheet: U2

Commit message: major work done. outline finished
Parts:
- removed J14: USB_C_Receptacle_USB2.0, Connector_USB:USB_C_Receptacle_HRO_TYPE-C-31-M-12, symbol Connector:USB_C_Receptacle_USB2.0
Changed lines of the file:
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@@
     (company "bastardkb")
   )
-  (junction (at -123.19 54.61) (diameter 0) (color 0 0 0 0)
-  )
   (junction (at 46.99 127) (diameter 0) (color 0 0 0 0)
   )
@@
   (junction (at 154.94 38.1) (diameter 0) (color 0 0 0 0)
   )
+  (junction (at -87.63 50.8) (diameter 0) (color 0 0 0 0)
+  )
   (junction (at 162.56 38.1) (diameter 0) (color 0 0 0 0)
   )
@@
   (junction (at 40.005 172.72) (diameter 0) (color 0 0 0 0)
   )
-  (junction (at -85.09 48.26) (diameter 0) (color 0 0 0 0)
-  )
-  (junction (at -111.76 72.39) (diameter 0) (color 0 0 0 0)
-  )
   (junction (at 157.48 38.1) (diameter 0) (color 0 0 0 0)
   )
@@
   (junction (at 160.02 38.1) (diameter 0) (color 0 0 0 0)
   )
+  (junction (at -87.63 48.26) (diameter 0) (color 0 0 0 0)
+  )
   (junction (at 33.02 113.03) (diameter 0) (color 0 0 0 0)
   )
@@
   (junction (at 154.94 144.78) (diameter 0) (color 0 0 0 0)
   )
-  (junction (at -104.14 72.39) (diameter 0) (color 0 0 0 0)
-  )
   (junction (at 198.12 106.68) (diameter 0) (color 0 0 0 0)
   )
@@
   (junction (at -68.58 40.64) (diameter 0) (color 0 0 0 0)
   )
-  (junction (at -123.19 49.53) (diameter 0) (color 0 0 0 0)
-  )
   (junction (at 130.81 185.42) (diameter 0) (color 0 0 0 0)
   )
   (junction (at 97.79 106.68) (diameter 0) (color 0 0 0 0)
   )
-  (junction (at -88.9 38.1) (diameter 0) (color 0 0 0 0)
-  )
   (junction (at 33.02 115.57) (diameter 0) (color 0 0 0 0)
   )
-  (junction (at -85.09 50.8) (diameter 0) (color 0 0 0 0)
-  )
   (junction (at 243.84 119.38) (diameter 0) (color 0 0 0 0)
   )
   (junction (at 29.845 29.845) (diameter 0) (color 0 0 0 0)
-  )
-  (junction (at -88.9 40.64) (diameter 0) (color 0 0 0 0)
   )
   (junction (at 143.51 38.1) (diameter 0) (color 0 0 0 0)
@@
     (stroke (width 0) (type default))
   )
-  (wire (pts (xy -123.19 49.53) (xy -85.09 49.53))
-    (stroke (width 0) (type default))
-  )
-  (wire (pts (xy -123.19 41.91) (xy -88.9 41.91))
-    (stroke (width 0) (type default))
-  )
   (wire (pts (xy 101.6 175.26) (xy 110.49 175.26))
     (stroke (width 0) (type default))
@@
     (stroke (width 0) (type default))
   )
-  (wire (pts (xy -111.76 81.28) (xy -111.76 72.39))
-    (stroke (width 0) (type default))
-  )
-  (wire (pts (xy -88.9 50.8) (xy -85.09 50.8))
+  (wire (pts (xy -88.9 50.8) (xy -87.63 50.8))
     (stroke (width 0) (type default))
   )
@@
     (stroke (width 0) (type default))
   )
-  (wire (pts (xy -85.09 54.61) (xy -85.09 50.8))
-    (stroke (width 0) (type default))
-  )
   (wire (pts (xy 267.97 137.16) (xy 256.54 137.16))
     (stroke (width 0) (type default))
@@
     (stroke (width 0) (type default))
   )
-  (wire (pts (xy -138.43 72.39) (xy -138.43 77.47))
-    (stroke (width 0) (type default))
-  )
   (wire (pts (xy 48.895 29.845) (xy 52.705 29.845))
     (stroke (width 0) (type default))
@@
     (stroke (width 0) (type default))
   )
-  (wire (pts (xy -88.9 39.37) (xy -88.9 38.1))
-    (stroke (width 0) (type default))
-  )
-  (wire (pts (xy -85.09 48.26) (xy -88.9 48.26))
-    (stroke (width 0) (type default))
-  )
   (polyline (pts (xy -39.37 137.795) (xy -121.92 137.795))
     (stroke (width 0) (type default))
@@
     (stroke (width 0) (type default))
   )
-  (wire (pts (xy -88.9 45.72) (xy -86.36 45.72))
-    (stroke (width 0) (type default))
-  )
   (wire (pts (xy 93.98 90.17) (xy 93.98 104.14))
     (stroke (width 0) (type default))
@@
     (stroke (width 0) (type default))
   )
-  (wire (pts (xy -86.36 45.72) (xy -85.09 48.26))
+  (wire (pts (xy -88.9 45.72) (xy -87.63 48.26))
     (stroke (width 0) (type default))
   )
@@
     (stroke (width 0) (type default))
   )
-  (wire (pts (xy -123.19 29.21) (xy -86.36 29.21))
-    (stroke (width 0) (type default))
-  )
   (wire (pts (xy 182.88 109.22) (xy 191.77 109.22))
     (stroke (width 0) (type default))
@@
     (stroke (width 0) (type default))
   )
-  (wire (pts (xy -85.09 49.53) (xy -85.09 48.26))
-    (stroke (width 0) (type default))
-  )
   (wire (pts (xy 175.26 40.64) (xy 175.26 38.1))
     (stroke (width 0) (type default))
   )
-  (wire (pts (xy -146.05 72.39) (xy -146.05 81.28))
+  (wire (pts (xy -87.63 48.26) (xy -88.9 48.26))
     (stroke (width 0) (type default))
   )
@@
     (stroke (width 0) (type default))
   )
-  (wire (pts (xy -88.9 41.91) (xy -88.9 40.64))
-    (stroke (width 0) (type default))
-  )
   (wire (pts (xy 58.42 113.03) (xy 58.42 118.11))
     (stroke (width 0) (type default))
@@
     (stroke (width 0) (type default))
   )
-  (wire (pts (xy -123.19 52.07) (xy -123.19 54.61))
-    (stroke (width 0) (type default))
-  )
-  (wire (pts (xy -123.19 54.61) (xy -85.09 54.61))
-    (stroke (width 0) (type default))
-  )
   (wire (pts (xy 148.59 175.26) (xy 157.48 175.26))
     (stroke (width 0) (type default))
@@
     (stroke (width 0) (type default))
   )
-  (wire (pts (xy -146.05 81.28) (xy -111.76 81.28))
-    (stroke (width 0) (type default))
-  )
   (wire (pts (xy 82.55 184.15) (xy 82.55 186.69))
     (stroke (width 0) (type default))
@@
     (stroke (width 0) (type default))
   )
-  (wire (pts (xy -123.19 39.37) (xy -88.9 39.37))
-    (stroke (width 0) (type default))
-  )
   (wire (pts (xy 97.79 105.41) (xy 97.79 106.68))
     (stroke (width 0) (type default))
@@
     (stroke (width 0) (type default))
   )
-  (wire (pts (xy -123.19 34.29) (xy -123.19 29.21))
-    (stroke (width 0) (type default))
-  )
   (wire (pts (xy 97.79 96.52) (xy 101.6 96.52))
     (stroke (width 0) (type default))
@@
     (stroke (width 0) (type default))
   )
-  (wire (pts (xy -138.43 77.47) (xy -104.14 77.47))
-    (stroke (width 0) (type default))
-  )
   (wire (pts (xy 91.44 184.15) (xy 91.44 186.69))
     (stroke (width 0) (type default))
@@
     (stroke (width 0) (type default))
   )
-  (wire (pts (xy -104.14 72.39) (xy -104.14 77.47))
-    (stroke (width 0) (type default))
-  )
   (polyline (pts (xy 77.47 194.31) (xy 172.72 194.31))
     (stroke (width 0) (type default))
@@
     (stroke (width 0) (type default))
   )
+  (wire (pts (xy -87.63 50.8) (xy -79.375 50.8))
+    (stroke (width 0) (type default))
+  )
   (wire (pts (xy 111.76 83.82) (xy 116.84 83.82))
     (stroke (width 0) (type default))
@@
     (stroke (width 0) (type default))
   )
-  (wire (pts (xy -85.09 50.8) (xy -86.36 53.34))
+  (wire (pts (xy -87.63 50.8) (xy -88.9 53.34))
     (stroke (width 0) (type default))
   )
@@
     (stroke (width 0) (type default))
   )
-  (wire (pts (xy -85.09 48.26) (xy -79.375 48.26))
-    (stroke (width 0) (type default))
-  )
   (wire (pts (xy 138.43 40.64) (xy 138.43 38.1))
     (stroke (width 0) (type default))
@@
     (stroke (width 0) (type default))
   )
-  (wire (pts (xy -123.19 46.99) (xy -123.19 49.53))
-    (stroke (width 0) (type default))
-  )
   (wire (pts (xy 182.88 134.62) (xy 191.77 134.62))
     (stroke (width 0) (type default))
@@
     (stroke (width 0) (type default))
   )
-  (wire (pts (xy -86.36 53.34) (xy -88.9 53.34))
-    (stroke (width 0) (type default))
-  )
   (wire (pts (xy 110.49 176.53) (xy 110.49 175.26))
     (stroke (width 0) (type default))
   )
-  (wire (pts (xy -85.09 50.8) (xy -79.375 50.8))
-    (stroke (width 0) (type default))
-  )
   (wire (pts (xy 157.48 184.15) (xy 157.48 185.42))
     (stroke (width 0) (type default))
@@
   )
   (wire (pts (xy 182.88 71.12) (xy 191.77 71.12))
+    (stroke (width 0) (type default))
+  )
+  (wire (pts (xy -87.63 48.26) (xy -79.375 48.26))
     (stroke (width 0) (type default))
   )
@@
     (effects (font (size 1.27 1.27)) (justify left bottom))
   )
-  (label "Gnd_daughter" (at -104.14 73.66 0) (fields_autoplaced)
+  (label "Gnd_daughter" (at -104.14 72.39 0) (fields_autoplaced)
     (effects (font (size 1.27 1.27)) (justify left bottom))
   )
@@
         )
       )
-    )
-  )
-  (symbol (lib_id "Connector:USB_C_Receptacle_USB2.0") (at -138.43 49.53 0) (unit 1)
-    (in_bom yes) (on_board yes) (dnp no) (fields_autoplaced)
-    (property "Reference" "J14" (at -138.43 26.67 0)
-      (effects (font (size 1.27 1.27)))
-    )
-    (property "Value" "USB_C_Receptacle_USB2.0" (at -138.43 29.21 0)
-      (effects (font (size 1.27 1.27)))
-    )
-    (property "Footprint" "Connector_USB:USB_C_Receptacle_HRO_TYPE-C-31-M-12" (at -134.62 49.53 0)
-      (effects (font (size 1.27 1.27)) hide)
-    )
-    (property "Datasheet" "https://www.usb.org/sites/default/files/documents/usb_type-c.zip" (at -134.62 49.53 0)
-      (effects (font (size 1.27 1.27)) hide)
-    )
-    (property "LCSC" "C223907" (at -138.43 49.53 0)
-      (effects (font (size 1.27 1.27)) hide)
-    )
-    (pin "A1")
-    (pin "A12")
-    (pin "A4")
-    (pin "A5")
-    (pin "A6")
-    (pin "A7")
-    (pin "A8")
-    (pin "A9")
-    (pin "B1")
-    (pin "B12")
-    (pin "B4")
-    (pin "B5")
-    (pin "B6")
-    (pin "B7")
-    (pin "B8")
-    (pin "B9")
-    (pin "S1")
-    (instances
-      (project "splinktegrated"
-        (path "/7353e96a-343a-4876-b497-b1d205a14d97"
-          (reference "J14") (unit 1)
-        )
-      )

Commit message: USB daugherboard
Parts:
- removed D2: B5817, Diode_SMD:D_SOD-323, symbol Device:D_Schottky
- removed F1: Polyfuse, Fuse:Fuse_0603_1608Metric, symbol Device:Polyfuse
- removed FB1: FerriteBead_Small, Inductor_SMD:L_0603_1608Metric, symbol Device:FerriteBead_Small
- removed J1: USB_C_Receptacle_USB2.0, Connector_USB:USB_C_Receptacle_HRO_TYPE-C-31-M-12, symbol Connector:USB_C_Receptacle_USB2.0
- removed J12, J2, J3, J4: Conn_01x04_Female, drawings:PinHeader_1x04_P2.54mm_Vertical, symbol Connector:Conn_01x04_Female
- removed R4, R5: 5.1k, Resistor_SMD:R_0402_1005Metric, symbol Device:R
- removed U4: USBLC6-2P6, Package_TO_SOT_SMD:SOT-666, symbol Power_Protection:USBLC6-2P6
- added D10, D11, D12, D13, D2, D3, D4, D5, D6, D7, D8, D9: D_Schottky_x2_KCom_AAK, customs:TSOT-23_HandSoldering, symbol Device:D_Schottky_x2_KCom_AAK
- added H1, H2, H3: MountingHole, MountingHole:MountingHole_2.2mm_M2, symbol Mechanical:MountingHole
- added H4: MountingHole_Pad, MountingHole:MountingHole_2.2mm_M2_Pad, symbol Mechanical:MountingHole_Pad
- added J1: X1224WRS-04-LPV01, locallib:PicoEZMate-Reinforced-Alt, symbol Connector_Generic_MountingPin:Conn_01x04_MountingPin
- added SW10, SW11, SW12, SW13, SW14, SW15, SW16, SW17, SW18, SW19, SW20, SW21, SW22, SW23, SW24, SW25, SW26, SW3, SW4, SW5, SW6, SW7, SW8, SW9: SW_Push, custom:SW_MX_reversible, symbol Switch:SW_Push
Connections:
- net VBUS is gone; now on net +5V: R10.2
- net +5V: now also J1.1 (Pin_1)
- net D+: now also J1.2 (Pin_2)
- net D-: now also J1.3 (Pin_3)
- net GND: now also H4.1, J1.4 (Pin_4), J1.MP (MountPin)
- new net: D3.1 (A), SW6.2
- new net: D3.2 (A), SW5.2
- new net: D4.1 (A), SW8.2
- new net: D4.2 (A), SW7.2
- new net: D10.1 (A), SW20.2
- new net: D6.1 (A), SW12.2
- new net: D7.1 (A), SW14.2
- new net: D7.2 (A), SW13.2
- new net: D6.2 (A), SW11.2
- new net: D11.1 (A), SW22.2
- new net: D12.2 (A), SW23.2
- new net: D9.2 (A), SW17.2
- new net: D8.2 (A), SW15.2
- new net: D12.1 (A), SW24.2
- new net: D13.2 (A), SW25.2
- new net: D10.2 (A), SW19.2
- new net: D5.1 (A), SW10.2
- new net: D5.2 (A), SW9.2
- new net: D8.1 (A), SW16.2
- new net: D2.1 (A), SW4.2
- new net: D2.2 (A), SW3.2
- new net: D9.1 (A), SW18.2
- new net: D11.2 (A), SW21.2
- new net: D13.1 (A), SW26.2
- new net col1: D2.3 (K), D3.3 (K)
- new net col2: D4.3 (K), D5.3 (K)
- new net col3: D6.3 (K), D7.3 (K)
- new net col4: D8.3 (K), D9.3 (K)
- new net col5: D10.3 (K), D11.3 (K)
- new net col6: D12.3 (K), D13.3 (K)
- new net row1: SW11.1, SW15.1, SW19.1, SW23.1, SW3.1, SW7.1
- new net row2: SW12.1, SW16.1, SW20.1, SW24.1, SW4.1, SW8.1
- new net row3: SW13.1, SW17.1, SW21.1, SW25.1, SW5.1, SW9.1
- new net row4: SW10.1, SW14.1, SW18.1, SW22.1, SW26.1, SW6.1
- no-connect marks 12 -> 10
Other:
- note removed: "ESD protection"
- note removed: "Headers"
- note removed: "USB-C connector"
- moved on the sheet: R10
